Commit message: Fix_nav2_error_slam

File: testpublicsher/src/my_bot/description/robot_config.xacro (robot description, xacro)
@@ -12,5 +12,5 @@
      <!--bottom_vaccum-->
     <joint name="bottom_joint" type="fixed">
-        <parent link="base_link"/>
+        <parent link="base_footprint"/>
         <child link="main_link"/>
         <origin xyz="0 0 ${wheel_radius}"/>

File: testpublicsher/src/my_bot/description/ros2_control.xacro (robot description, xacro)
@@ -25,4 +25,8 @@
         <plugin name="gazebo_ros2_control" filename="libgazebo_ros2_control.so">
             <parameters>$(find my_bot)/config/my_controller.yaml</parameters>
+                <!-- <ros>
+                    <argument>~/out:=keyboard</argument>
+                </ros>
+                <output_type>geometry_msgs/msg/Twist</output_type> -->
         </plugin>
     </gazebo>
